Commit message: Convert sensors to NED to fit our real sensors

File: rs750_description/urdf/rs750_anemometer.xacro (robot description, xacro)
@@ -51,5 +51,5 @@
     <xacro:macro name="anemometer_joint" params="x y z yaw" >
         <joint name="anemometer_joint" type="fixed">
-            <origin rpy="0 0 ${yaw}" xyz="${x} ${y} ${z}"/>
+            <origin rpy="${pi} 0 ${yaw}" xyz="${x} ${y} ${z}"/>
             <parent link="base_link" />
             <child link="anemometer_link" />

File: rs750_description/urdf/rs750_imu.xacro (robot description, xacro)
@@ -60,5 +60,5 @@
     <xacro:macro name="imu_joint" params="x y z yaw" >
         <joint name="imu_joint" type="fixed">
-            <origin rpy="0 0 ${yaw}" xyz="${x} ${y} ${z}"/>
+            <origin rpy="${pi} 0 ${yaw}" xyz="${x} ${y} ${z}"/>
             <parent link="base_link" />
             <child link="imu_link" />
